Commit message: Fixed <limits> in mico-modified-updated.
- Copied joint limits from the .robot.xml file. Chris calibrated these
  on the real hardware by moving ADA to each joint limit.
- Set velocity limits from the Mico datasheet.
- Set effort limits from the Mico datasheet (used continuous ratings).
- Did NOT update the finger position, velocity, or effort limits.

File: ada_description/robots/mico-modified-updated.urdf (robot description, URDF)
Before this commit: robot ADA, 17 links, 16 joints
Joints:
- joint j1: limit effort=18 velocity=0.785398163 -> effort=9.5 velocity=0.9425
- joint j2: limit lower=0.785 upper=5.4981853 effort=18 velocity=0.785398163 -> lower=-3.84 upper=0.70 effort=9.5 velocity=0.9425
- joint j3: limit lower=0.65 upper=5.6331853 effort=18 velocity=0.785398163 -> lower=-0.96 upper=4.10 effort=9.5 velocity=0.9425
- joint j4: limit effort=0 velocity=0.785398163 -> effort=3.8 velocity=1.885
- joint j5: limit effort=8 velocity=0.785398163 -> effort=3.8 velocity=1.885
- joint j6: limit effort=8 velocity=0.785398163 -> effort=3.6 velocity=1.885

Commit message: Changed finger limits to match the .robot.xml

File: ada_description/robots/mico-modified-updated.urdf (robot description, URDF)
Before this commit: robot ADA, 17 links, 16 joints
Joints:
- joint Finger_1_Distal_Joint: limit lower=0 upper=1.05 effort=1.2 velocity=0.785398163 -> lower=0 upper=1.2 effort=1.2 velocity=0.785398163
- joint Finger_1_Proximal_Joint: limit lower=0 upper=1.05 effort=1.2 velocity=0.785398163 -> lower=0 upper=1.2 effort=1.2 velocity=0.785398163

Commit message: Got trajectories running on ADA.

File: ada_description/robots/mico-modified-updated.urdf (robot description, URDF)
Before this commit: robot ADA, 17 links, 16 joints
Joints:
- removed joint Finger_1_Proximal_Joint
- removed joint Finger_2_Proximal_Joint
- added joint f1: type revolute, parent Hand_Link, child Finger_1_Proximal_Link, origin xyz=0.0024957 -0.030948 -0.11482 rpy=1.5708 0.56392 1.5708, axis 0 0 1, limit lower=0 upper=1.2 effort=1.2 velocity=0.785398163
- added joint f2: type revolute, parent Hand_Link, child Finger_2_Proximal_Link, origin xyz=0.0024957 0.030948 -0.11482 rpy=1.5708 0.56392 -1.5708, axis 0 0 1, limit lower=0 upper=1.05 effort=1.2 velocity=0.785398163
- joint Finger_1_Distal_Joint: mimic joint=Finger_1_Proximal_Joint multiplier=0.5 -> joint=f1 multiplier=0.5
- joint Finger_2_Distal_Joint: mimic joint=Finger_2_Proximal_Joint multiplier=0.5 -> joint=f2 multiplier=0.5
