Commit message: moved mico-modified to use mesh with softkinetic camera

File: ada_description/robots/mico-modified.urdf (robot description, URDF)
Before this commit: robot ADA, 17 links, 16 joints
Links:
- link Hand_Link: geometry collision mesh filename=package://ada_description/meshes/Hand_Link_camera.STL; visual mesh filename=package://ada_description/meshes/Hand_Link_camera.STL

Commit message: Updated with limits from specs

File: ada_description/robots/mico-modified.urdf (robot description, URDF)
Before this commit: robot ADA, 17 links, 16 joints
Joints:
- joint j1: limit effort=18 velocity=0.785398163 -> effort=18 velocity=0.94
- joint j2: limit lower=0.785 upper=5.4981853 effort=18 velocity=0.785398163 -> lower=0.785 upper=5.4981853 effort=18 velocity=0.94
- joint j3: limit lower=0.65 upper=5.6331853 effort=18 velocity=0.785398163 -> lower=0.65 upper=5.6331853 effort=18 velocity=0.94
- joint j4: limit effort=0 velocity=0.785398163 -> effort=0 velocity=2.0
- joint j5: limit effort=8 velocity=0.785398163 -> effort=8 velocity=2.0
- joint j6: limit effort=8 velocity=0.785398163 -> effort=8 velocity=2.0

Commit message: Modified robot limits for the fingers, to allow tighter grips

File: ada_description/robots/mico-modified.urdf (robot description, URDF)
Before this commit: robot ADA, 17 links, 16 joints
Joints:
- joint f1: limit lower=0 upper=1.05 effort=1.2 velocity=0.785398163 -> lower=0 upper=1.20 effort=1.2 velocity=0.785398163
- joint f2: limit lower=0 upper=1.05 effort=1.2 velocity=0.785398163 -> lower=0 upper=1.20 effort=1.2 velocity=0.785398163

Commit message: Fixed joint-limits

File: ada_description/robots/mico-modified.urdf (robot description, URDF)
Before this commit: robot ADA, 17 links, 16 joints
Joints:
- joint j1: limit effort=18 velocity=0.94 -> effort=18 velocity=0.942
- joint j2: limit lower=0.785 upper=5.4981853 effort=18 velocity=0.94 -> lower=0.785 upper=5.4981853 effort=18 velocity=0.942
- joint j3: limit lower=0.65 upper=5.6331853 effort=18 velocity=0.94 -> lower=0.65 upper=5.6331853 effort=18 velocity=0.942
- joint j4: limit effort=0 velocity=2.0 -> effort=0 velocity=1.884
- joint j5: limit effort=8 velocity=2.0 -> effort=8 velocity=1.884
- joint j6: limit effort=8 velocity=2.0 -> effort=8 velocity=1.884

Commit message: Updated joint limits in mico-modified.

File: ada_description/robots/mico-modified.urdf (robot description, URDF)
Before this commit: robot ADA, 17 links, 16 joints
Joints:
- joint j1: limit effort=18 velocity=0.942 -> effort=9.5 velocity=0.9425
- joint j2: limit lower=0.785 upper=5.4981853 effort=18 velocity=0.942 -> lower=0.785 upper=5.4981853 effort=9.5 velocity=0.9425
- joint j3: limit lower=0.65 upper=5.6331853 effort=18 velocity=0.942 -> lower=0.65 upper=5.6331853 effort=9.5 velocity=0.9425
- joint j4: limit effort=0 velocity=1.884 -> effort=3.8 velocity=1.885
- joint j5: limit effort=8 velocity=1.884 -> effort=3.8 velocity=1.885
- joint j6: limit effort=8 velocity=1.884 -> effort=3.6 velocity=1.885

Commit message: Fixed mico-modified mimic joints.

File: ada_description/robots/mico-modified.urdf (robot description, URDF)
Before this commit: robot ADA, 17 links, 16 joints
Joints:
- removed joint Finger_1_Distal_Joint
- removed joint Finger_2_Distal_Joint
- added joint f1_distal: type revolute, parent Finger_1_Proximal_Link, child Finger_1_Distal_Link, origin xyz=-0.003 -0.044 0 rpy=0 0 -0.19199, axis 0 0 1, limit lower=0 upper=1.05 effort=1.2 velocity=0.785398163, mimic joint=f1 multiplier=0.5
- added joint f2_distal: type revolute, parent Finger_2_Proximal_Link, child Finger_2_Distal_Link, origin xyz=-0.003 -0.044 0 rpy=0 0 -0.19199, axis 0 0 1, limit lower=0 upper=1.05 effort=1.2 velocity=0.785398163, mimic joint=f2 multiplier=0.5
