Commit message: content for weight_expressiveness

File: ada_description/robots/mico-modified2.urdf (robot description, URDF)
Before this commit: robot ADA, 17 links, 16 joints
Joints:
- joint f1: limit lower=0 upper=1.10 effort=1.2 velocity=0.785398163 -> lower=0 upper=1.20 effort=1.2 velocity=0.785398163
