Commit message: modified jaco end effector to match ada

File: ada_description/robots/jaco.urdf (robot description, URDF)
Before this commit: robot JACO, 15 links, 14 joints
Joints:
- joint j2n6a300_end_effector_offset: origin xyz=0 0 -0.1600 rpy=3.14159265359 0 0 -> xyz=0 0 0.000 rpy=0 0 1.570795

Commit message: added fake camera and more configs

File: ada_description/robots/jaco.urdf (robot description, URDF)
Before this commit: robot JACO, 15 links, 14 joints
Links:
- added link Camera_Depth_Frame, mass 0.05
- added link Camera_RGB_Frame, mass 0.05
Joints:
- added joint Camera_Depth_Joint: type fixed, parent Camera_Depth_Frame, child Camera_RGB_Frame, origin xyz=0.045 -0.015 -0.03 rpy=0 0.000 0
- added joint Camera_Joint: type fixed, parent j2n6a300_link_6, child Camera_Depth_Frame, origin xyz=-0.047 0.05 -0.090  rpy=-2.92 0.000 0
