Commit message: Fixed joint limits in URDF.

File: ada_description/robots/mico.urdf (robot description, URDF)
Before this commit: robot ADA, 17 links, 16 joints
Joints:
- joint f1: limit lower=0 upper=1.20 effort=1.2 velocity=0.785398163 -> lower=0 upper=1.33555556 effort=1.2 velocity=0.785398163
- joint f2: limit lower=0 upper=1.20 effort=1.2 velocity=0.785398163 -> lower=0 upper=1.33555556 effort=1.2 velocity=0.785398163
- joint j2: limit lower=0.785 upper=5.4981853 effort=9.5 velocity=0.9425 -> lower=-3.84517851 upper=0.62658588 effort=9.5 velocity=0.9425
- joint j3: limit lower=0.65 upper=5.6331853 effort=9.5 velocity=0.9425 -> lower=-0.95864778 upper=4.1040905 effort=9.5 velocity=0.9425

Commit message: Fixed joint limits on fingers.

File: ada_description/robots/mico.urdf (robot description, URDF)
Before this commit: robot ADA, 17 links, 16 joints
Joints:
- joint f1: limit lower=0 upper=1.33555556 effort=1.2 velocity=0.785398163 -> lower=-0.01 upper=1.33555556 effort=1.2 velocity=0.785398163
- joint f2: limit lower=0 upper=1.33555556 effort=1.2 velocity=0.785398163 -> lower=-0.01 upper=1.33555556 effort=1.2 velocity=0.785398163

Commit message: Tweaked finger joint limits.

File: ada_description/robots/mico.urdf (robot description, URDF)
Before this commit: robot ADA, 17 links, 16 joints
Joints:
- joint f1: limit lower=-0.01 upper=1.33555556 effort=1.2 velocity=0.785398163 -> lower=-0.01 upper=1.35 effort=1.2 velocity=0.785398163
- joint f2: limit lower=-0.01 upper=1.33555556 effort=1.2 velocity=0.785398163 -> lower=-0.01 upper=1.35 effort=1.2 velocity=0.785398163

Commit message: changes in the mico.urdf

File: ada_description/robots/mico.urdf (robot description, URDF)
Before this commit: robot ADA, 17 links, 16 joints
Links:
- added link Camera_RGB_Frame, mass 0.05
Joints:
- added joint Camera_Joint: type fixed, parent Hand_Link, child Camera_RGB_Frame, origin xyz=0.048 0.014 -0.089  rpy=-2.969 0.001 -1.572

Commit message: added configurations and changed mico.urdf file

File: ada_description/robots/mico.urdf (robot description, URDF)
Before this commit: robot ADA, 18 links, 17 joints
Joints:
- joint Camera_Joint: origin xyz=0.048 0.014 -0.089  rpy=-2.969 0.001 -1.572 -> xyz=0.047 0.05 -0.090  rpy=-2.92 0.000 -1.571

Commit message: added slight rotation to j2 to bring it in line with reality

File: ada_description/robots/mico.urdf (robot description, URDF)
Before this commit: robot ADA, 18 links, 17 joints
Joints:
- joint j2: origin xyz=0 -0.00175 0.11875 rpy=1.5708 0 3.1416 -> xyz=0 -0.00175 0.11875 rpy=1.5708 -0.22 3.1416

Commit message: Reduced velocity limits to 0.75 rad/s.

File: ada_description/robots/mico.urdf (robot description, URDF)
Before this commit: robot ADA, 18 links, 17 joints
Joints:
- joint j1: limit effort=9.5 velocity=0.9425 -> effort=9.5 velocity=0.75
- joint j2: limit lower=-3.84517851 upper=0.62658588 effort=9.5 velocity=0.9425 -> lower=-3.84517851 upper=0.62658588 effort=9.5 velocity=0.75
- joint j3: limit lower=-0.95864778 upper=4.1040905 effort=9.5 velocity=0.9425 -> lower=-0.95864778 upper=4.1040905 effort=9.5 velocity=0.75
- joint j4: limit effort=3.8 velocity=1.885 -> effort=3.8 velocity=0.75
- joint j5: limit effort=3.8 velocity=1.885 -> effort=3.8 velocity=0.75
- joint j6: limit effort=3.6 velocity=1.885 -> effort=3.6 velocity=0.75

Commit message: changed urdf joint offset because of Kinova's upgrade

File: ada_description/robots/mico.urdf (robot description, URDF)
Before this commit: robot ADA, 18 links, 17 joints
Joints:
- joint j2: origin xyz=0 -0.00175 0.11875 rpy=1.5708 -0.22 3.1416 -> xyz=0 -0.00175 0.11875 rpy=1.5708 0.0 3.1416

Commit message: URDF and model files released with kinova driver

File: ada_description/robots/mico.urdf (robot description, URDF)
Before this commit: robot ADA, 18 links, 17 joints
Links:
- removed link Arm_Link
- removed link Arm_Ring_Link
- removed link Camera_RGB_Frame
- removed link Finger_1_Distal_Link
- removed link Finger_1_Proximal_Link
- removed link Finger_2_Distal_Link
- removed link Finger_2_Proximal_Link
- removed link Forearm_Link
- removed link Forearm_Ring_Link
- removed link Hand_Link
- removed link Hand_Ring_Link
- removed link Shoulder_Link
- removed link Shoulder_Ring_Link
- removed link Wrist_1_Link
- removed link Wrist_1_Ring_Link
- removed link Wrist_2_Link
- removed link Wrist_2_Ring_Link
- removed link base_link
- added link mico_end_effector
- added link mico_link_1, mass 0.825; collision mesh filename=package://ada_description/meshes/mico_link_1.dae; visual mesh filename=package://ada_description/meshes/mico_link_1.dae
- added link mico_link_2, mass 1.215; collision mesh filename=package://ada_description/meshes/mico_link_2.dae; visual mesh filename=package://ada_description/meshes/mico_link_2.dae
- added link mico_link_3, mass 0.775; collision mesh filename=package://ada_description/meshes/mico_link_3.dae; visual mesh filename=package://ada_description/meshes/mico_link_3.dae
- added link mico_link_4, mass 0.415; collision mesh filename=package://ada_description/meshes/mico_link_4.dae; visual mesh filename=package://ada_description/meshes/mico_link_4.dae
- added link mico_link_5, mass 0.415; collision mesh filename=package://ada_description/meshes/mico_link_4.dae; visual mesh filename=package://ada_description/meshes/mico_link_4.dae
- added link mico_link_base, mass 1.000; collision mesh filename=package://ada_description/meshes/mico_link_base.dae; visual mesh filename=package://ada_description/meshes/mico_link_base.dae
- added link mico_link_finger_1, mass 0.010; collision mesh filename=package://ada_description/meshes/finger_proximal_limb_1.dae; visual mesh filename=package://ada_description/meshes/finger_proximal_limb_1.dae
- added link mico_link_finger_2, mass 0.010; collision mesh filename=package://ada_description/meshes/finger_proximal_limb_1.dae; visual mesh filename=package://ada_description/meshes/finger_proximal_limb_1.dae
- added link mico_link_finger_tip_1, mass 0.010; collision mesh filename=package://ada_description/meshes/finger_distal_limb_1.dae; visual mesh filename=package://ada_description/meshes/finger_distal_limb_1.dae
- added link mico_link_finger_tip_2, mass 0.010; collision mesh filename=package://ada_description/meshes/finger_distal_limb_1.dae; visual mesh filename=package://ada_description/meshes/finger_distal_limb_1.dae
- added link mico_link_hand, mass 0.557; collision mesh filename=package://ada_description/meshes/mico_link_hand.dae; visual mesh filename=package://ada_description/meshes/mico_link_hand.dae
- added link world
Joints:
- removed joint Arm_Ring_Joint
- removed joint Camera_Joint
- removed joint Forearm_Ring_Joint
- removed joint Hand_Ring_Joint
- removed joint Shoulder_Ring_Joint
- removed joint Wrist_1_Ring_Joint
- removed joint Wrist_2_Ring_Joint
- removed joint f1
- removed joint f1_distal
- removed joint f2
- removed joint f2_distal
- removed joint j1
- removed joint j2
- removed joint j3
- removed joint j4
- removed joint j5
- removed joint j6
- added joint mico_joint_1: type continuous, parent mico_link_base, child mico_link_1, origin xyz=0 0 0.1535 rpy=3.14159265359 0 3.14159265359, axis 0 0 -1, limit effort=30 velocity=0.35
- added joint mico_joint_2: type revolute, parent mico_link_1, child mico_link_2, origin xyz=0 0 -0.1185 rpy=-1.57079632679 3.14159265359 0, axis 0 0 1, limit lower=-3.14159265359 upper=0.0 effort=30 velocity=0.35
- added joint mico_joint_3: type revolute, parent mico_link_2, child mico_link_3, origin xyz=0.29 0 0 rpy=3.14159265359 0 1.57079632679, axis 0 0 -1, limit lower=-3.92699081699 upper=0.785398163397 effort=30 velocity=0.35
- added joint mico_joint_4: type continuous, parent mico_link_3, child mico_link_4, origin xyz=0.123 0 -0.00845 rpy=3.14159265359 1.57079632679 0, axis 0 0 -1, limit effort=30 velocity=0.35
- added joint mico_joint_5: type continuous, parent mico_link_4, child mico_link_5, origin xyz=0.037 0 -0.06408 rpy=0 -1.0471975512 0, axis 0 0 -1, limit effort=30 velocity=0.35
- added joint mico_joint_6: type continuous, parent mico_link_5, child mico_link_hand, origin xyz=0.037 0 -0.06408 rpy=-1.0471975512 0 1.57079632679, axis 0 0 -1, limit effort=30 velocity=0.35
- added joint mico_joint_finger_1: type revolute, parent mico_link_hand, child mico_link_finger_1, origin xyz=-0.03095 -0.0025 -0.116 rpy=1.57079632679 1.57079632679 0, axis 0 0 1, limit lower=0 upper=0.698131700798 effort=30 velocity=5
- added joint mico_joint_finger_2: type revolute, parent mico_link_hand, child mico_link_finger_2, origin xyz=0.03095 -0.0025 -0.116 rpy=-1.57079632679 1.57079632679 0, axis 0 0 1, limit lower=0 upper=0.698131700798 effort=30 velocity=5
- added joint mico_joint_finger_tip_1: type fixed, parent mico_link_finger_1, child mico_link_finger_tip_1, origin xyz=0.035 -0.0295 -0.0025 rpy=0 0 0, axis 0 0 1
- added joint mico_joint_finger_tip_2: type fixed, parent mico_link_finger_2, child mico_link_finger_tip_2, origin xyz=0.035 -0.0295 -0.0025 rpy=0 0 0, axis 0 0 1
- added joint mico_link_hand_to_end_effector: type fixed, parent mico_link_hand, child mico_end_effector, origin xyz=0 0 -0.1687 rpy=0 3.14159265359 0
- added joint world_2_base_fixed: type fixed, parent world, child mico_link_base, origin xyz=0 0 0 rpy=0 0 0

Commit message: More realistic joint limits for joints 2 and 3

File: ada_description/robots/mico.urdf (robot description, URDF)
Before this commit: robot ADA, 13 links, 12 joints
Joints:
- joint mico_joint_2: limit lower=-3.14159265359 upper=0.0 effort=30 velocity=0.35 -> lower=-3.8451785 upper=0.7035858 effort=30 velocity=0.35
- joint mico_joint_3: limit lower=-3.92699081699 upper=0.785398163397 effort=30 velocity=0.35 -> lower=-4.104090 upper=0.95768524 effort=30 velocity=0.35

Commit message: editting urdf to render correctly

File: ada_description/robots/mico.urdf (robot description, URDF)
Before this commit: robot ADA, 18 links, 17 joints
Links:
- link Hand_Link: geometry collision mesh filename=package://ada_description/meshes/Hand_Link.STL; visual mesh filename=package://ada_description/meshes/Hand_Link.STL

Commit message: code used currently for mutual adaptation

File: ada_description/robots/mico.urdf (robot description, URDF)
Before this commit: robot ADA, 18 links, 17 joints
Links:
- removed link Finger_1_Distal_Link
- removed link Finger_1_Proximal_Link
- removed link Finger_2_Distal_Link
- removed link Finger_2_Proximal_Link
Joints:
- removed joint f1
- removed joint f1_distal
- removed joint f2
- removed joint f2_distal

Commit message: set finger limits back

File: ada_description/robots/mico.urdf (robot description, URDF)
Before this commit: robot ADA, 13 links, 12 joints
Joints:
- joint mico_joint_finger_1: limit lower=0 upper=0.698131700798 effort=30 velocity=5 -> lower=0 upper=1.35 effort=30 velocity=5
- joint mico_joint_finger_2: limit lower=0 upper=0.698131700798 effort=30 velocity=5 -> lower=0 upper=1.35 effort=30 velocity=5

Commit message: Changed to map not world

File: ada_description/robots/mico.urdf (robot description, URDF)
Before this commit: robot ADA, 13 links, 12 joints
Links:
- removed link world
- added link map
Joints:
- removed joint world_2_base_fixed
- added joint map_2_base_fixed: type fixed, parent map, child mico_link_base, origin xyz=0 0 0 rpy=0 0 0

Commit message: Updated mico.urdf with old velocity limits

File: ada_description/robots/mico.urdf (robot description, URDF)
Before this commit: robot ADA, 13 links, 12 joints
Joints:
- joint mico_joint_1: limit effort=30 velocity=0.35 -> effort=30 velocity=0.9425
- joint mico_joint_2: limit lower=-3.8451785 upper=0.7035858 effort=30 velocity=0.35 -> lower=-3.8451785 upper=0.7035858 effort=30 velocity=0.9425
- joint mico_joint_3: limit lower=-4.104090 upper=0.95768524 effort=30 velocity=0.35 -> lower=-4.104090 upper=0.95768524 effort=30 velocity=0.9425
- joint mico_joint_4: limit effort=30 velocity=0.35 -> effort=30 velocity=1.885
- joint mico_joint_5: limit effort=30 velocity=0.35 -> effort=30 velocity=1.885
- joint mico_joint_6: limit effort=30 velocity=0.35 -> effort=30 velocity=1.885
- joint mico_joint_finger_1: limit lower=0 upper=1.35 effort=30 velocity=5 -> lower=0 upper=1.35 effort=30 velocity=0.785398163
- joint mico_joint_finger_2: limit lower=0 upper=1.35 effort=30 velocity=5 -> lower=0 upper=1.35 effort=30 velocity=0.785398163

Commit message: added camera transform

File: ada_description/robots/mico.urdf (robot description, URDF)
Before this commit: robot ADA, 13 links, 12 joints
Links:
- added link Camera_RGB_Frame, mass 0.05
Joints:
- added joint Camera_Joint: type fixed, parent mico_link_hand, child Camera_RGB_Frame, origin xyz=-0.047 0.05 -0.090  rpy=-2.92 0.000 0

Commit message: Change urdf to use hand model with camera

File: ada_description/robots/mico.urdf (robot description, URDF)
Before this commit: robot ADA, 14 links, 13 joints
Links:
- link mico_link_hand: geometry collision mesh filename=package://ada_description/meshes/mico_hand_structureio.dae; visual mesh filename=package://ada_description/meshes/mico_hand_structureio.dae

Commit message: stick on camera stl

File: ada_description/robots/mico.urdf (robot description, URDF)
Before this commit: robot ADA, 14 links, 13 joints
Links:
- added link Camera_Collision_Frame, mass 0.05
- link Camera_RGB_Frame: geometry collision mesh filename=package://ada_description/meshes/StructureIO.stl; visual mesh filename=package://ada_description/meshes/StructureIO.stl
- link mico_link_hand: geometry collision mesh filename=package://ada_description/meshes/mico_link_hand.dae; visual mesh filename=package://ada_description/meshes/mico_link_hand.dae
Joints:
- added joint Camera_Collision_Joint: type fixed, parent mico_link_hand, child Camera_Collision_Frame, origin xyz=0 0 0 rpy=0 0 0

Commit message: switch back to dae

File: ada_description/robots/mico.urdf (robot description, URDF)
Before this commit: robot ADA, 15 links, 14 joints
Links:
- link Camera_RGB_Frame: geometry collision mesh filename=package://ada_description/meshes/structureio.dae; visual mesh filename=package://ada_description/meshes/structureio.dae

Commit message: Aligned camera

File: ada_description/robots/mico.urdf (robot description, URDF)
Before this commit: robot ADA, 15 links, 14 joints
Links:
- link Camera_RGB_Frame: geometry collision mesh filename=package://ada_description/meshes/StructureIO.stl; visual mesh filename=package://ada_description/meshes/StructureIO.stl

Commit message: Rotated camera mesh to be on correct side of hand.

File: ada_description/robots/mico.urdf (robot description, URDF)
Before this commit: robot ADA, 15 links, 14 joints
Links:
- link Camera_Collision_Frame: geometry collision mesh filename=package://ada_description/meshes/StructureIO.stl; visual mesh filename=package://ada_description/meshes/StructureIO.stl
- link Camera_RGB_Frame: geometry 

Commit message: reentered  fingers

File: ada_description/robots/mico.urdf (robot description, URDF)
Before this commit: robot ADA, 14 links, 13 joints
Links:
- added link Finger_1_Distal_Link, mass 0.0121939815401302; collision mesh filename=package://ada_description/meshes/Finger_1_Distal_Link.STL; visual mesh filename=package://ada_description/meshes/Finger_1_Distal_Link.STL
- added link Finger_1_Proximal_Link, mass 0.0106365590225629; collision mesh filename=package://ada_description/meshes/Finger_1_Proximal_Link.STL; visual mesh filename=package://ada_description/meshes/Finger_1_Proximal_Link.STL
- added link Finger_2_Distal_Link, mass 0.0121939010456702; collision mesh filename=package://ada_description/meshes/Finger_2_Distal_Link.STL; visual mesh filename=package://ada_description/meshes/Finger_2_Distal_Link.STL
- added link Finger_2_Proximal_Link, mass 0.0106364391584646; collision mesh filename=package://ada_description/meshes/Finger_2_Proximal_Link.STL; visual mesh filename=package://ada_description/meshes/Finger_2_Proximal_Link.STL
Joints:
- added joint f1: type revolute, parent Hand_Link, child Finger_1_Proximal_Link, origin xyz=0.0024957 -0.030948 -0.11482 rpy=1.5708 0.56392 1.5708, axis 0 0 1, limit lower=-0.01 upper=1.35 effort=1.2 velocity=0.785398163
- added joint f1_distal: type revolute, parent Finger_1_Proximal_Link, child Finger_1_Distal_Link, origin xyz=-0.003 -0.044 0 rpy=0 0 -0.19199, axis 0 0 1, limit lower=0 upper=1.05 effort=1.2 velocity=0.785398163, mimic joint=f1 multiplier=0.5
- added joint f2: type revolute, parent Hand_Link, child Finger_2_Proximal_Link, origin xyz=0.0024957 0.030948 -0.11482 rpy=1.5708 0.56392 -1.5708, axis 0 0 1, limit lower=-0.01 upper=1.35 effort=1.2 velocity=0.785398163
- added joint f2_distal: type revolute, parent Finger_2_Proximal_Link, child Finger_2_Distal_Link, origin xyz=-0.003 -0.044 0 rpy=0 0 -0.19199, axis 0 0 1, limit lower=0 upper=1.05 effort=1.2 velocity=0.785398163, mimic joint=f2 multiplier=0.5
- joint j2: origin xyz=0 -0.00175 0.11875 rpy=1.5708 0.0 3.1416 -> xyz=0 -0.00175 0.11875 rpy=1.5708 0 3.1416

Commit message: recalibrated velocity limits

File: ada_description/robots/mico.urdf (robot description, URDF)
Before this commit: robot ADA, 14 links, 13 joints
Joints:
- joint mico_joint_1: limit effort=30 velocity=0.9425 -> effort=30 velocity=0.84
- joint mico_joint_2: limit lower=-3.8451785 upper=0.7035858 effort=30 velocity=0.9425 -> lower=-3.8451785 upper=0.7035858 effort=30 velocity=0.8425
- joint mico_joint_3: limit lower=-4.104090 upper=0.95768524 effort=30 velocity=0.9425 -> lower=-4.104090 upper=0.95768524 effort=30 velocity=0.83
- joint mico_joint_4: limit effort=30 velocity=1.885 -> effort=30 velocity=0.84
- joint mico_joint_5: limit effort=30 velocity=1.885 -> effort=30 velocity=0.84
- joint mico_joint_6: limit effort=30 velocity=1.885 -> effort=30 velocity=0.84

Commit message: created textured mesh for structureio

File: ada_description/robots/mico.urdf (robot description, URDF)
Before this commit: robot ADA, 15 links, 14 joints
Links:
- link Camera_Collision_Frame: geometry collision mesh filename=package://ada_description/meshes/StructureIO.stl; visual mesh filename=package://ada_description/meshes/structureio.dae

Commit message: added urdf frames. switched color and depth

File: ada_description/robots/mico.urdf (robot description, URDF)
Before this commit: robot ADA, 15 links, 14 joints
Links:
- added link Camera_Depth_Frame, mass 0.05
Joints:
- added joint Camera_Depth_Joint: type fixed, parent Camera_Depth_Frame, child Camera_RGB_Frame, origin xyz=0.045 -0.015 -0.03 rpy=0 0.000 0
- joint Camera_Joint: child Camera_RGB_Frame -> Camera_Depth_Frame

Commit message: just added astra for collision. Need to update Camera_Depth_Frame

File: ada_description/robots/mico.urdf (robot description, URDF)
Before this commit: robot ADA, 16 links, 15 joints
Links:
- link Camera_Collision_Frame: geometry collision mesh filename=package://ada_description/meshes/astra.stl; visual mesh filename=package://ada_description/meshes/astra.stl
Joints:
- joint Camera_Collision_Joint: origin xyz=0 0 0 rpy=0 0 0 -> xyz=0 0 -0.004 rpy=0 3.14159 0

Commit message: approximate depth frame translation

File: ada_description/robots/mico.urdf (robot description, URDF)
Before this commit: robot ADA, 16 links, 15 joints
Joints:
- joint Camera_Joint: origin xyz=-0.047 0.05 -0.090  rpy=-2.92 0.000 0 -> xyz=-0.042 0.073 -0.104 rpy=0.0 0.000 0

Commit message: measured astra RGB frame added

File: ada_description/robots/mico.urdf (robot description, URDF)
Before this commit: robot ADA, 16 links, 15 joints
Joints:
- removed joint Camera_Depth_Joint
- added joint Camera_RGB_Joint: type fixed, parent mico_link_hand, child Camera_RGB_Frame, origin xyz=-0.0135 0.0725 -0.104 rpy=0.18375 0.000 0

Commit message: Updated RGB and Depth frames to be consistant with StructureIO

File: ada_description/robots/mico.urdf (robot description, URDF)
Before this commit: robot ADA, 16 links, 15 joints
Joints:
- joint Camera_Joint: origin xyz=-0.042 0.073 -0.104 rpy=0.0 0.000 0 -> xyz=-0.042 0.073 -0.104 rpy=-2.9578426535897933 0.000 0
- joint Camera_RGB_Joint: origin xyz=-0.0135 0.0725 -0.104 rpy=0.18375 0.000 0 -> xyz=-0.0135 0.0725 -0.104 rpy=-2.9578426535897933 0.000 0
